File: pico-rom-emu.kicad_sch (KiCad schematic)
At the start: 37 parts, among them J1 HDR_28C256, J2 HDR_UART, J4 HDR_SWD, Q1 MMBT2222A, SW1 SW_Push, U1 74HCT574D, U2 74HCT574D, U3 74HCT574D, U4 74HCT08, U5 RaspberryPi_Pico2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

Commit message: pre rev1 order
Parts:
- H1, H2, H3, H4: now not fitted
- J1: value HDR_28C256 -> N3440-5302RB
Connections:
- net LADH: now also U5.25 (GPIO19); no longer U5.26 (GPIO20)
- net LADL: now also U5.26 (GPIO20); no longer U5.25 (GPIO19)
- net XDA0: now also U5.17 (GPIO13); no longer U5.9 (GPIO6)
- net XDA1: now also U5.16 (GPIO12); no longer U5.10 (GPIO7)
- net XDA2: now also U5.15 (GPIO11); no longer U5.11 (GPIO8)
- net XDA3: now also U5.14 (GPIO10); no longer U5.12 (GPIO9)
- net XDA4: now also U5.9 (GPIO6); no longer U5.14 (GPIO10)
- net XDA5: now also U5.10 (GPIO7); no longer U5.15 (GPIO11)
- net XDA6: now also U5.11 (GPIO8); no longer U5.16 (GPIO12)
- net XDA7: now also U5.12 (GPIO9); no longer U5.17 (GPIO13)
Changed lines of the file:
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@@
 		(rev "1")
 		(company "Grackle Computing")
+		(comment 1 "CC BY-SA-NC 4.0")
 	)
 	(rectangle
@@
 	(text "ROM Control\nSharing Logic"
 		(exclude_from_sim no)
-		(at 195.58 86.36 0)
+		(at 196.85 88.9 0)
 		(effects
 			(font
@@
 	(wire
 		(pts
-			(xy 128.27 86.36) (xy 148.59 86.36)
+			(xy 128.27 86.36) (xy 146.05 86.36)
 		)
 		(stroke
@@
 	(wire
 		(pts
-			(xy 83.82 83.82) (xy 146.05 83.82)
+			(xy 83.82 83.82) (xy 148.59 83.82)
 		)
 		(stroke
@@
 	(wire
 		(pts
-			(xy 148.59 86.36) (xy 148.59 128.27)
-		)
-		(stroke
-			(width 0)
-			(type default)
-		)
-	)
-	(wire
-		(pts
 			(xy 35.56 59.69) (xy 35.56 60.96)
 		)
@@
 	(wire
 		(pts
+			(xy 148.59 83.82) (xy 148.59 128.27)
+		)
+		(stroke
+			(width 0)
+			(type default)
+		)
+	)
+	(wire
+		(pts
 			(xy 251.46 46.99) (xy 256.54 46.99)
 		)
@@
 		)
 	)
-	(wire
-		(pts
-			(xy 146.05 83.82) (xy 146.05 125.73)
-		)
-		(stroke
-			(width 0)
-			(type default)
-		)
-	)
 	(bus
 		(pts
@@
 	(wire
 		(pts
+			(xy 146.05 86.36) (xy 146.05 125.73)
+		)
+		(stroke
+			(width 0)
+			(type default)
+		)
+	)
+	(wire
+		(pts
 			(xy 104.14 35.56) (xy 106.68 35.56)
 		)
@@
 	)
 	(label "LADL"
-		(at 140.97 125.73 180)
+		(at 140.97 128.27 180)
 		(effects
 			(font
@@
 	)
 	(label "XDA4"
-		(at 82.55 140.97 0)
+		(at 82.55 130.81 0)
 		(effects
 			(font
@@
 	)
 	(label "XDA5"
-		(at 82.55 143.51 0)
+		(at 82.55 133.35 0)
 		(effects
 			(font
@@
 	)
 	(label "XDA2"
-		(at 82.55 135.89 0)
+		(at 82.55 143.51 0)
 		(effects
 			(font
@@
 	)
 	(label "XDA3"
-		(at 82.55 138.43 0)
+		(at 82.55 140.97 0)
 		(effects
 			(font
@@
 	)
 	(label "XDA1"
-		(at 82.55 133.35 0)
+		(at 82.55 146.05 0)
 		(effects
 			(font
@@
 	)
 	(label "XDA7"
-		(at 82.55 148.59 0)
+		(at 82.55 138.43 0)
 		(effects
 			(font
@@
 	)
 	(label "XDA0"
-		(at 82.55 130.81 0)
+		(at 82.55 148.59 0)
 		(effects
 			(font
@@
 	)
 	(label "XDA6"
-		(at 82.55 146.05 0)
+		(at 82.55 135.89 0)
 		(effects
 			(font
@@
 	)
 	(label "LADH"
-		(at 140.97 128.27 180)
+		(at 140.97 125.73 180)
 		(effects
 			(font
@@
 		(exclude_from_sim yes)
 		(in_bom no)
-		(on_board yes)
-		(dnp no)
+		(on_board no)
+		(dnp yes)
 		(fields_autoplaced yes)
 		(property "Reference" "H4"
@@
 	(symbol
 		(lib_id "Graphic:Logo_Open_Hardware_Small")
-		(at 196.85 173.99 0)
+		(at 213.36 173.99 0)
 		(unit 1)
 		(exclude_from_sim yes)
@@
 		(fields_autoplaced yes)
 		(property "Reference" "#SYM1"
-			(at 196.85 167.005 0)
+			(at 213.36 167.005 0)
 			(effects
 				(font
@@
 		)
 		(property "Value" "Logo_Open_Hardware_Small"
-			(at 196.85 179.705 0)
+			(at 213.36 179.705 0)
 			(effects
 				(font
@@
 		)
 		(property "Footprint" "Symbol:OSHW-Symbol_8.9x8mm_Copper"
-			(at 196.85 173.99 0)
+			(at 213.36 173.99 0)
 			(effects
 				(font
@@
 		)
 		(property "Datasheet" "~"
-			(at 196.85 173.99 0)
+			(at 213.36 173.99 0)
 			(effects
 				(font
@@
 		)
 		(property "Description" "Open Hardware logo, small"
-			(at 196.85 173.99 0)
+			(at 213.36 173.99 0)
 			(effects
 				(font
@@
 			)
 		)
-		(property "Value" "HDR_28C256"
+		(property "Value" "N3440-5302RB"
 			(at 245.11 70.866 0)
 			(effects
@@
 		(exclude_from_sim yes)
 		(in_bom no)
-		(on_board yes)
-		(dnp no)
+		(on_board no)
+		(dnp yes)
 		(fields_autoplaced yes)
 		(property "Reference" "H1"
@@
 	(symbol
 		(lib_id "GrackleLogo12mm:LOGO")
-		(at 184.15 173.99 0)
+		(at 184.15 171.45 0)
 		(unit 1)
 		(exclude_from_sim no)
@@
 		(fields_autoplaced yes)
 		(property "Reference" "#G1"
-			(at 184.15 168.6237 0)
+			(at 184.15 166.0837 0)
 			(effects
 				(font
@@
 		)
 		(property "Value" "GrackleComputing"
-			(at 184.15 179.3563 0)
+			(at 184.15 176.8163 0)
 			(effects
 				(font
@@
 		)
 		(property "Footprint" "CustomSymbols:GrackleLogo12mm"
-			(at 184.15 173.99 0)
+			(at 184.15 171.45 0)
 			(effects
 				(font
@@
 		)
 		(property "Datasheet" ""
-			(at 184.15 173.99 0)
+			(at 184.15 171.45 0)
 			(effects
 				(font
@@
 		)
 		(property "Description" ""
-			(at 184.15 173.99 0)
+			(at 184.15 171.45 0)
 			(effects
 				(font
@@
 		(exclude_from_sim yes)
 		(in_bom no)
-		(on_board yes)
-		(dnp no)
+		(on_board no)
+		(dnp yes)
 		(fields_autoplaced yes)
 		(property "Reference" "H3"
@@
 		(exclude_from_sim yes)
 		(in_bom no)
-		(on_board yes)
-		(dnp no)
+		(on_board no)
+		(dnp yes)
 		(fields_autoplaced yes)
 		(property "Reference" "H2"

Commit message: rev 1 pre-production clean up
Parts:
- R1: value 1k8 -> 270R; Mfr ERJ-P06J182V -> CRGCQ0805F270R
- R2: value 680R -> 620R; Mfr ERJ-P06J182V -> CRCW0805620RFKEA
- R3: value 680R -> 620R; Mfr ERJ-UP6D6800V -> CRCW0805620RFKEA
- R4: value 3k3 -> 4k7; Mfr ERJ-P06D3301V -> CR0805-FX-4701ELF
- R5: value 1k8 -> 620R; Mfr ERJ-P06J182V -> CRCW0805620RFKEA
- R6: value 680R -> 270R; Mfr ERJ-UP6D6800V -> CRGCQ0805F270R
- R8: Mfr ERJ-P06D3301V -> CRCW080510R0FKEAHP
- R9: value 1k8 -> 120R; Mfr ERJ-P06J182V -> ERJ-P06F1200V
- U5: Mfr (none) -> SC1631
Other:
- note added: "- 74HCT series logic used to allow 3.3v -> 5v logic without discrete level shifting circuitry. - x~{RST} signal is open-drain, Q1 prevents sinking DUT reset signal current with MCU. - Remove F2 if current draw exceeds DUT supply capability."
- note removed: "- 74HCT series logic used to allow 3.3v -> 5v logic without discrete level shifting circuitry. - x~{RST} signal is open-drain, Q1 prevents sinking DUT reset signal current with MCU."
- moved on the sheet: C5, C6, D6, F1, F2, H1, H2, H3, H4, R4, U4D, U4E
